File: CSD95379Q3M-BDBB-BB.kicad_sch (KiCad schematic)
At the start: 23 parts, among them U101 CSD97394Q4M, U102 CSD97394Q4M, U103 INA260, U104 INA260

Commit message: Route some more stuff, move things a bit.
Connections:
- net ~{SKIP}-B: now reaches U102.1 (~{SKIP})
- net PWM-B: now reaches U102.8 (PWM)
- net ~{SKIP}-A: now reaches U101.1 (~{SKIP})
- net PWM-A: now reaches U101.8 (PWM)
Changed lines of the file:
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@@
   (junction (at 112.395 97.79) (diameter 0) (color 0 0 0 0)
   )
+  (junction (at 165.735 69.215) (diameter 0) (color 0 0 0 0)
+  )
   (junction (at 127.635 81.915) (diameter 0) (color 0 0 0 0)
   )
@@
   (junction (at 78.105 111.125) (diameter 0) (color 0 0 0 0)
   )
-  (junction (at 160.02 69.215) (diameter 0) (color 0 0 0 0)
-  )
   (junction (at 92.075 69.215) (diameter 0) (color 0 0 0 0)
   )
@@
     (stroke (width 0) (type default))
   )
+  (wire (pts (xy 49.53 73.025) (xy 66.675 73.025))
+    (stroke (width 0) (type default))
+  )
   (wire (pts (xy 88.265 121.92) (xy 90.805 121.92))
     (stroke (width 0) (type default))
@@
     (stroke (width 0) (type default))
   )
-  (wire (pts (xy 160.02 62.23) (xy 160.02 69.215))
+  (wire (pts (xy 165.735 62.23) (xy 165.735 69.215))
     (stroke (width 0) (type default))
   )
@@
     (stroke (width 0) (type default))
   )
+  (wire (pts (xy 49.53 75.565) (xy 66.675 75.565))
+    (stroke (width 0) (type default))
+  )
   (wire (pts (xy 156.845 127) (xy 161.925 127))
     (stroke (width 0) (type default))
@@
     (stroke (width 0) (type default))
   )
+  (wire (pts (xy 158.115 75.565) (xy 174.625 75.565))
+    (stroke (width 0) (type default))
+  )
   (wire (pts (xy 128.905 132.08) (xy 128.905 134.62))
     (stroke (width 0) (type default))
@@
     (stroke (width 0) (type default))
   )
-  (wire (pts (xy 160.02 69.215) (xy 158.115 69.215))
-    (stroke (width 0) (type default))
-  )
   (wire (pts (xy 165.735 70.485) (xy 165.735 69.215))
     (stroke (width 0) (type default))
   )
+  (wire (pts (xy 158.115 73.025) (xy 174.625 73.025))
+    (stroke (width 0) (type default))
+  )
   (wire (pts (xy 136.525 132.08) (xy 133.985 132.08))
     (stroke (width 0) (type default))
   )
-  (wire (pts (xy 95.885 132.08) (xy 104.14 132.08))
+  (wire (pts (xy 95.885 132.08) (xy 107.315 132.08))
     (stroke (width 0) (type default))
   )
@@
     (stroke (width 0) (type default))
   )
+  (wire (pts (xy 158.115 69.215) (xy 165.735 69.215))
+    (stroke (width 0) (type default))
+  )
   (wire (pts (xy 87.63 111.125) (xy 90.805 111.125))
     (stroke (width 0) (type default))
   )
-  (wire (pts (xy 165.735 69.215) (xy 160.02 69.215))
-    (stroke (width 0) (type default))
-  )
   (wire (pts (xy 150.495 59.055) (xy 151.765 59.055))
     (stroke (width 0) (type default))
@@
   (label "VAS" (at 94.615 121.92 0) (fields_autoplaced)
     (effects (font (size 1.27 1.27)) (justify left bottom))
+  )
+  (label "PWM-A" (at 49.53 75.565 180) (fields_autoplaced)
+    (effects (font (size 1.27 1.27)) (justify right bottom))
   )
   (label "VBS" (at 130.175 121.92 180) (fields_autoplaced)
@@
     (effects (font (size 1.27 1.27)) (justify right bottom))
   )
-  (label "VA" (at 104.14 132.08 0) (fields_autoplaced)
+  (label "VA" (at 107.315 132.08 0) (fields_autoplaced)
+    (effects (font (size 1.27 1.27)) (justify left bottom))
+  )
+  (label "~{SKIP}-A" (at 49.53 73.025 180) (fields_autoplaced)
+    (effects (font (size 1.27 1.27)) (justify right bottom))
+  )
+  (label "PWM-B" (at 174.625 75.565 0) (fields_autoplaced)
     (effects (font (size 1.27 1.27)) (justify left bottom))
   )
   (label "VBS" (at 126.365 69.215 180) (fields_autoplaced)
     (effects (font (size 1.27 1.27)) (justify right bottom))
+  )
+  (label "~{SKIP}-B" (at 174.625 73.025 0) (fields_autoplaced)
+    (effects (font (size 1.27 1.27)) (justify left bottom))
   )
   (netclass_flag "" (length 2.54) (shape round) (at 59.69 69.215 90) (fields_autoplaced)
@@
     )
   )
-  (symbol (lib_id "power:+5V") (at 160.02 62.23 0) (unit 1)
-    (in_bom yes) (on_board yes) (dnp no) (fields_autoplaced)
-    (property "Reference" "#PWR0101" (at 160.02 66.04 0)
-      (effects (font (size 1.27 1.27)) hide)
-    )
-    (property "Value" "+5V" (at 160.02 57.15 0)
+  (symbol (lib_id "power:+5V") (at 165.735 62.23 0) (unit 1)
+    (in_bom yes) (on_board yes) (dnp no) (fields_autoplaced)
+    (property "Reference" "#PWR0101" (at 165.735 66.04 0)
+      (effects (font (size 1.27 1.27)) hide)
+    )
+    (property "Value" "+5V" (at 165.735 57.15 0)
       (effects (font (size 1.27 1.27)))
     )
-    (property "Footprint" "" (at 160.02 62.23 0)
-      (effects (font (size 1.27 1.27)) hide)
-    )
-    (property "Datasheet" "" (at 160.02 62.23 0)
-      (effects (font (size 1.27 1.27)) hide)
-    )
+    (property "Footprint" "" (at 165.735 62.23 0)
+      (effects (font (size 1.27 1.27)) hide)
+    )
+    (property "Datasheet" "" (at 165.735 62.23 0)
+      (effects (font (size 1.27 1.27)) hide)
+    )

Commit message: Fixed a net name.
Connections:
- net VAS: no longer L101.1, U101.4 (VSW)
- new net VSWA: L101.1, U101.4 (VSW)
Changed lines of the file:
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@@
     (effects (font (size 1.27 1.27)) (justify left bottom))
   )
-  (label "VSWB" (at 128.27 74.295 0) (fields_autoplaced)
+  (label "VSWB" (at 120.015 74.295 0) (fields_autoplaced)
     (effects (font (size 1.27 1.27)) (justify left bottom))
   )
-  (label "VSWA" (at 92.075 74.295 0) (fields_autoplaced)
+  (label "VSWA" (at 99.695 74.295 0) (fields_autoplaced)
     (effects (font (size 1.27 1.27)) (justify left bottom))
   )
